File: hardware/rp2350_zero_carrier/rp2350_zero_carrier.kicad_sch (KiCad schematic)
At the start: 12 parts, among them J1 RP2350-Zero_Header(23pin,GPIO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, J2 USB-A_Host(Neltron_5075AR-04-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, J3 RP2350-Zero_Header(23pin,ボード2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, SW1 1回路2接点スイッチ(3pin,NKK_115643,ON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, SW2 1回路2接点スイッチ(3pin,NKK_115643,ON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, SW3 1回路2接点スイッチ(3pin,NKK_115643,ON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, SW4 1回路2接点スイッチ(3pin,NKK_115643,ON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, SW5 1回路2接点スイッチ(3pin,NKK_115643,ON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, SW6 タクトスイッチ4pin(Akizuki_DTS-63-N-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

Commit message: wip(hardware): add USB VBUS protection circuit
Parts:
- added CIN: 1uF X7R 16V, rp2350_zero_carrier:C_0603, symbol Device:C
- added R_FAULT: 100k, rp2350_zero_carrier:R_0603, symbol Device:R
- added R_ILIM: 52.3k 1%, rp2350_zero_carrier:R_0603, symbol Device:R
- added U1: TPS2553DBVR, rp2350_zero_carrier:TPS2553DBVR, symbol TPS2553DBVR
Connections:
- net GND: now also CIN.1, R_ILIM.1, U1.2 (GND)
- net VBUS_USB_A: now also U1.6 (OUT); no longer F1.1 (Pin_1)
- new net TPS_ILIM: R_ILIM.2, U1.5 (ILIM)
- new net USB_PWR_FAULT_N: R_FAULT.2, U1.4 (FAULT)
- new net VBUS_TPS_IN: CIN.2, F1.1 (Pin_1), R_FAULT.1, U1.1 (IN), U1.3 (EN)
Changed lines of the file:
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@@
     )
   )
+  (symbol (lib_id "TPS2553DBVR") (at 228.6 203.2 0) (unit 1)
+    (in_bom yes) (on_board yes) (dnp no) (fields_autoplaced yes)
+    (property "Reference" "U1" (at 228.6 197.74 0) (effects (font (size 1.27 1.27))))
+    (property "Value" "TPS2553DBVR" (at 228.6 208.66 0) (effects (font (size 1.27 1.27))))
+    (property "Footprint" "rp2350_zero_carrier:TPS2553DBVR" (at 228.6 203.2 0) (effects (font (size 1.27 1.27)) hide))
+    (property "Datasheet" "https://www.ti.com/lit/ds/symlink/tps2553.pdf" (at 228.6 203.2 0) (effects (font (size 1.27 1.27)) hide))
+    (pin "1")
+    (pin "2")
+    (pin "3")
+    (pin "4")
+    (pin "5")
+    (pin "6")
+    (instances
+      (project "rp2350_zero_carrier"
+        (path "/"
+          (reference "U1") (unit 1)
+        )
+      )
+    )
+  )
+  (symbol (lib_id "Device:C") (at 213.36 177.8 0) (unit 1)
+    (in_bom yes) (on_board yes) (dnp no) (fields_autoplaced yes)
+    (property "Reference" "CIN" (at 216.36 175.26 0) (effects (font (size 1.27 1.27))))
+    (property "Value" "1uF X7R 16V" (at 216.36 180.34 0) (effects (font (size 1.27 1.27))))
+    (property "Footprint" "rp2350_zero_carrier:C_0603" (at 213.36 177.8 0) (effects (font (size 1.27 1.27)) hide))
+    (property "Datasheet" "" (at 213.36 177.8 0) (effects (font (size 1.27 1.27)) hide))
+    (pin "1")
+    (pin "2")
+    (instances
+      (project "rp2350_zero_carrier"
+        (path "/"
+          (reference "CIN") (unit 1)
+        )
+      )
+    )
+  )
+  (symbol (lib_id "Device:R") (at 243.84 177.8 0) (unit 1)
+    (in_bom yes) (on_board yes) (dnp no) (fields_autoplaced yes)
+    (property "Reference" "R_ILIM" (at 251.84 175.26 0) (effects (font (size 1.27 1.27))))
+    (property "Value" "52.3k 1%" (at 251.84 180.34 0) (effects (font (size 1.27 1.27))))
+    (property "Footprint" "rp2350_zero_carrier:R_0603" (at 243.84 177.8 0) (effects (font (size 1.27 1.27)) hide))
+    (property "Datasheet" "" (at 243.84 177.8 0) (effects (font (size 1.27 1.27)) hide))
+    (pin "1")
+    (pin "2")
+    (instances
+      (project "rp2350_zero_carrier"
+        (path "/"
+          (reference "R_ILIM") (unit 1)
+        )
+      )
+    )
+  )
+  (symbol (lib_id "Device:R") (at 243.84 222.25 0) (unit 1)
+    (in_bom yes) (on_board yes) (dnp no) (fields_autoplaced yes)
+    (property "Reference" "R_FAULT" (at 251.84 219.71 0) (effects (font (size 1.27 1.27))))
+    (property "Value" "100k" (at 251.84 224.79 0) (effects (font (size 1.27 1.27))))
+    (property "Footprint" "rp2350_zero_carrier:R_0603" (at 243.84 222.25 0) (effects (font (size 1.27 1.27)) hide))
+    (property "Datasheet" "" (at 243.84 222.25 0) (effects (font (size 1.27 1.27)) hide))
+    (pin "1")
+    (pin "2")
+    (instances
+      (project "rp2350_zero_carrier"
+        (path "/"
+          (reference "R_FAULT") (unit 1)
+        )
+      )
+    )
+  )
+  (wire (pts (xy 223.52 205.74) (xy 220.98 205.74)) (stroke (width 0) (type default)) (uuid "b1c9a1a0-w001-4a00-9000-000000000001"))
+  (label "VBUS_TPS_IN" (at 220.98 205.74 0) (effects (font (size 1.27 1.27)) (justify right)) (uuid "b1c9a1a0-l001-4a00-9000-000000000001"))
+  (wire (pts (xy 223.52 203.2) (xy 220.98 203.2)) (stroke (width 0) (type default)) (uuid "b1c9a1a0-w002-4a00-9000-000000000001"))
+  (label "GND" (at 220.98 203.2 0) (effects (font (size 1.27 1.27)) (justify right)) (uuid "b1c9a1a0-l002-4a00-9000-000000000001"))
+  (wire (pts (xy 223.52 200.66) (xy 220.98 200.66)) (stroke (width 0) (type default)) (uuid "b1c9a1a0-w003-4a00-9000-000000000001"))
+  (label "VBUS_TPS_IN" (at 220.98 200.66 0) (effects (font (size 1.27 1.27)) (justify right)) (uuid "b1c9a1a0-l003-4a00-9000-000000000001"))
+  (wire (pts (xy 233.68 200.66) (xy 236.22 200.66)) (stroke (width 0) (type default)) (uuid "b1c9a1a0-w004-4a00-9000-000000000001"))
+  (label "VBUS_USB_A" (at 236.22 200.66 0) (effects (font (size 1.27 1.27)) (justify left)) (uuid "b1c9a1a0-l004-4a00-9000-000000000001"))
+  (wire (pts (xy 233.68 203.2) (xy 236.22 203.2)) (stroke (width 0) (type default)) (uuid "b1c9a1a0-w005-4a00-9000-000000000001"))
+  (label "TPS_ILIM" (at 236.22 203.2 0) (effects (font (size 1.27 1.27)) (justify left)) (uuid "b1c9a1a0-l005-4a00-9000-000000000001"))
+  (wire (pts (xy 233.68 205.74) (xy 236.22 205.74)) (stroke (width 0) (type default)) (uuid "b1c9a1a0-w006-4a00-9000-000000000001"))
+  (label "USB_PWR_FAULT_N" (at 236.22 205.74 0) (effects (font (size 1.27 1.27)) (justify left)) (uuid "b1c9a1a0-l006-4a00-9000-000000000001"))
+  (wire (pts (xy 213.36 181.61) (xy 213.36 184.15)) (stroke (width 0) (type default)) (uuid "b1c9a1a0-w007-4a00-9000-000000000001"))
+  (label "VBUS_TPS_IN" (at 213.36 184.15 0) (effects (font (size 1.27 1.27)) (justify left)) (uuid "b1c9a1a0-l007-4a00-9000-000000000001"))
+  (wire (pts (xy 213.36 173.99) (xy 213.36 171.45)) (stroke (width 0) (type default)) (uuid "b1c9a1a0-w008-4a00-9000-000000000001"))
+  (label "GND" (at 213.36 171.45 0) (effects (font (size 1.27 1.27)) (justify left)) (uuid "b1c9a1a0-l008-4a00-9000-000000000001"))
+  (wire (pts (xy 243.84 181.61) (xy 243.84 184.15)) (stroke (width 0) (type default)) (uuid "b1c9a1a0-w009-4a00-9000-000000000001"))
+  (label "TPS_ILIM" (at 243.84 184.15 0) (effects (font (size 1.27 1.27)) (justify left)) (uuid "b1c9a1a0-l009-4a00-9000-000000000001"))
+  (wire (pts (xy 243.84 173.99) (xy 243.84 171.45)) (stroke (width 0) (type default)) (uuid "b1c9a1a0-w010-4a00-9000-000000000001"))
+  (label "GND" (at 243.84 171.45 0) (effects (font (size 1.27 1.27)) (justify left)) (uuid "b1c9a1a0-l010-4a00-9000-000000000001"))
+  (wire (pts (xy 243.84 226.06) (xy 243.84 228.6)) (stroke (width 0) (type default)) (uuid "b1c9a1a0-w011-4a00-9000-000000000001"))
+  (label "USB_PWR_FAULT_N" (at 243.84 228.6 0) (effects (font (size 1.27 1.27)) (justify left)) (uuid "b1c9a1a0-l011-4a00-9000-000000000001"))
+  (wire (pts (xy 243.84 218.44) (xy 243.84 215.9)) (stroke (width 0) (type default)) (uuid "b1c9a1a0-w012-4a00-9000-000000000001"))
+  (label "VBUS_TPS_IN" (at 243.84 215.9 0) (effects (font (size 1.27 1.27)) (justify left)) (uuid "b1c9a1a0-l012-4a00-9000-000000000001"))
   (symbol (lib_id "Connector_Generic:Conn_01x04") (at 160 90 0) (unit 1)
     (in_bom yes) (on_board yes) (dnp no) (fields_autoplaced yes)
@@
   (label "USB_A_DM" (at 110 93.65 0) (effects (font (size 1.27 1.27)) (justify left)))
   (label "VBUS_5V" (at 102.38 81.27 0) (effects (font (size 1.27 1.27)) (justify right)))
-  (label "VBUS_USB_A" (at 102.38 78.73 0) (effects (font (size 1.27 1.27)) (justify right)))
+  (label "VBUS_TPS_IN" (at 102.38 78.73 0) (effects (font (size 1.27 1.27)) (justify right)))
   (label "VBUS_USB_A_SW" (at 152.38 93.81 0) (effects (font (size 1.27 1.27)) (justify right)))
   (label "USB_A_DM" (at 152.38 91.27 0) (effects (font (size 1.27 1.27)) (justify right)))

Commit message: checkpoint(hardware): refine USB VBUS protection layout
Parts:
- added COUT: 220uF 16V, rp2350_zero_carrier:CP_Radial_D6.3mm_P2.50mm, symbol Device:C_Polarized
Connections:
- net GND: now also COUT.2 (-)
- net VBUS_USB_A_SW: now also COUT.1 (+)
Changed lines of the file:
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@@
+    )
+  )
+  (symbol (lib_id "Device:C_Polarized") (at 269.24 177.8 0) (unit 1)
+    (in_bom yes) (on_board yes) (dnp no) (fields_autoplaced yes)
+    (property "Reference" "COUT" (at 272.24 175.26 0) (effects (font (size 1.27 1.27))))
+    (property "Value" "220uF 16V" (at 272.24 180.34 0) (effects (font (size 1.27 1.27))))
+    (property "Footprint" "rp2350_zero_carrier:CP_Radial_D6.3mm_P2.50mm" (at 269.24 177.8 0) (effects (font (size 1.27 1.27)) hide))
+    (property "Datasheet" "https://akizukidenshi.com/catalog/g/g110326/" (at 269.24 177.8 0) (effects (font (size 1.27 1.27)) hide))
+    (pin "1")
+    (pin "2")
+    (instances
+      (project "rp2350_zero_carrier"
+        (path "/"
+          (reference "COUT") (unit 1)
+        )
+      )
     )
   )
@@
   (wire (pts (xy 243.84 218.44) (xy 243.84 215.9)) (stroke (width 0) (type default)) (uuid "b1c9a1a0-w012-4a00-9000-000000000001"))
   (label "VBUS_TPS_IN" (at 243.84 215.9 0) (effects (font (size 1.27 1.27)) (justify left)) (uuid "b1c9a1a0-l012-4a00-9000-000000000001"))
+  (wire (pts (xy 269.24 173.99) (xy 269.24 171.45)) (stroke (width 0) (type default)) (uuid "c0a7b000-w001-4a00-9000-000000000001"))
+  (label "VBUS_USB_A_SW" (at 269.24 171.45 0) (effects (font (size 1.27 1.27)) (justify left)) (uuid "c0a7b000-l001-4a00-9000-000000000001"))
+  (wire (pts (xy 269.24 181.61) (xy 269.24 184.15)) (stroke (width 0) (type default)) (uuid "c0a7b000-w002-4a00-9000-000000000001"))
+  (label "GND" (at 269.24 184.15 0) (effects (font (size 1.27 1.27)) (justify left)) (uuid "c0a7b000-l002-4a00-9000-000000000001"))
   (symbol (lib_id "Connector_Generic:Conn_01x04") (at 160 90 0) (unit 1)
     (in_bom yes) (on_board yes) (dnp no) (fields_autoplaced yes)

Commit message: checkpoint(hardware): align schematic pin mapping with PCB
Parts:
- R2: footprint rp2350_zero_carrier:R_Axial_THT_P10.16mm -> rp2350_zero_carrier:R_Axial_THT_P10.16mm_notopsilk
Connections:
- net GND: now also J2.4 (Pin_4); no longer J2.1 (Pin_1)
- net GP12_USB_DP: now also R1.1; no longer J2.3 (Pin_3), R1.2, R2.1
- net GP13_USB_DM: now also J2.3 (Pin_3), R1.2, R2.1; no longer R2.2
- net VBUS_5V: now also F1.1 (Pin_1); no longer F1.2 (Pin_2)
- net VBUS_TPS_IN: now also F1.2 (Pin_2); no longer F1.1 (Pin_1)
- net VBUS_USB_A_SW: now also J2.1 (Pin_1); no longer J2.4 (Pin_4)
- net USB_A_DP renamed USB_A_DM
- net USB_A_DM: now also R2.2; no longer R1.1
Changed lines of the file:
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@@
     (property "Reference" "R2" (at 118 100 0) (effects (font (size 1.27 1.27))))
     (property "Value" "22" (at 118 106 0) (effects (font (size 1.27 1.27))))
-    (property "Footprint" "rp2350_zero_carrier:R_Axial_THT_P10.16mm" (at 110 100 0) (effects (font (size 1.27 1.27)) hide))
+    (property "Footprint" "rp2350_zero_carrier:R_Axial_THT_P10.16mm_notopsilk" (at 110 100 0) (effects (font (size 1.27 1.27)) hide))
     (property "Datasheet" "" (at 110 100 0) (effects (font (size 1.27 1.27)) hide))
     (pin "1")
@@
   (label "GP13_USB_DM" (at 32.38 110.95 0) (effects (font (size 1.27 1.27)) (justify right)))
   (label "GP12_USB_DP" (at 32.38 108.41 0) (effects (font (size 1.27 1.27)) (justify right)))
-  (label "GP12_USB_DP" (at 110 96.35 0) (effects (font (size 1.27 1.27)) (justify left)))
-  (label "USB_A_DP" (at 110 83.65 0) (effects (font (size 1.27 1.27)) (justify left)))
-  (label "GP13_USB_DM" (at 110 106.35 0) (effects (font (size 1.27 1.27)) (justify left)))
-  (label "USB_A_DM" (at 110 93.65 0) (effects (font (size 1.27 1.27)) (justify left)))
-  (label "VBUS_5V" (at 102.38 81.27 0) (effects (font (size 1.27 1.27)) (justify right)))
-  (label "VBUS_TPS_IN" (at 102.38 78.73 0) (effects (font (size 1.27 1.27)) (justify right)))
-  (label "VBUS_USB_A_SW" (at 152.38 93.81 0) (effects (font (size 1.27 1.27)) (justify right)))
-  (label "USB_A_DM" (at 152.38 91.27 0) (effects (font (size 1.27 1.27)) (justify right)))
-  (label "USB_A_DP" (at 152.38 88.73 0) (effects (font (size 1.27 1.27)) (justify right)))
-  (label "GND" (at 152.38 86.19 0) (effects (font (size 1.27 1.27)) (justify right)))
+  (label "USB_A_DP" (at 110 96.35 0) (effects (font (size 1.27 1.27)) (justify left)))
+  (label "GP12_USB_DP" (at 110 83.65 0) (effects (font (size 1.27 1.27)) (justify left)))
+  (label "USB_A_DM" (at 110 106.35 0) (effects (font (size 1.27 1.27)) (justify left)))
+  (label "GP13_USB_DM" (at 110 93.65 0) (effects (font (size 1.27 1.27)) (justify left)))
+  (label "VBUS_TPS_IN" (at 102.38 81.27 0) (effects (font (size 1.27 1.27)) (justify right)))
+  (label "VBUS_5V" (at 102.38 78.73 0) (effects (font (size 1.27 1.27)) (justify right)))
+  (label "GND" (at 152.38 93.81 0) (effects (font (size 1.27 1.27)) (justify right)))
+  (label "USB_A_DP" (at 152.38 91.27 0) (effects (font (size 1.27 1.27)) (justify right)))
+  (label "USB_A_DM" (at 152.38 88.73 0) (effects (font (size 1.27 1.27)) (justify right)))
+  (label "VBUS_USB_A_SW" (at 152.38 86.19 0) (effects (font (size 1.27 1.27)) (justify right)))
   (label "GP28_SW1_GAME_MODE" (at 50 23.65 90) (effects (font (size 1.27 1.27)) (justify right)))
   (label "GND" (at 52.54 36.35 90) (effects (font (size 1.27 1.27)) (justify left)))
